Commit message: 完善URDF机器人模型

File: src/my_first_pkg/urdf/my_robot.urdf (robot description, URDF)
Before this commit: robot my_robot, 5 links, 4 joints
Links:
- link base_link: geometry collision box size=0.3 0.2 0.1; visual box size=0.3 0.2 0.1
- link left_wheel: geometry collision cylinder length=0.03 radius=0.05; visual cylinder length=0.03 radius=0.05
- link right_wheel: geometry collision cylinder length=0.03 radius=0.05; visual cylinder length=0.03 radius=0.05

Commit message: 添加激光雷达传感器，发布/scan话题

File: src/my_first_pkg/urdf/my_robot.urdf (robot description, URDF)
Before this commit: robot my_robot, 5 links, 4 joints
Links:
- added link obstacle_box; collision box size=0.5 0.5 0.5; visual box size=0.5 0.5 0.5
Joints:
- added joint obstacle_joint: type fixed, parent base_footprint, child obstacle_box, origin xyz=2.0 0 0.25

Commit message: 添加雷达数据处理节点，实现障碍物检测

File: src/my_first_pkg/urdf/my_robot.urdf (robot description, URDF)
Before this commit: robot my_robot, 6 links, 5 joints
Links:
- removed link obstacle_box
Joints:
- removed joint obstacle_joint
